Commit message: Funcionamiento de mutt con GPS y con SLAM

File: src/mutt_robot/models/mutt/robot.xacro (robot description, xacro)
@@ -19,7 +19,7 @@
   <xacro:property name="camera_y" value="0.00"/>
   <xacro:property name="camera_z" value="0.75"/>
-  <xacro:property name="lidar_x" value="-0.50"/>
+  <xacro:property name="lidar_x" value="1.0"/>
   <xacro:property name="lidar_y" value="0.00"/>
-  <xacro:property name="lidar_z" value="1.40"/>
+  <xacro:property name="lidar_z" value="1.30"/>
   <xacro:property name="imu_x" value="-0.50"/>
   <xacro:property name="imu_y" value="0.20"/>
